File: pinebook-pro-3v3sys.kicad_pcb (KiCad board)
At the start: 2 copper layers, 7.8 x 17.9 mm, 23 parts, among them J1 Conn_01x03, J2 Conn_02x03_Counter_Clockwise, J3 Conn_01x01, J4 Conn_01x03, J5 Conn_01x01, U1 TPS63806

Commit message: Add components for mousebites
Parts:
- removed REF** (x4): Mousebite_0.3mm, Mousebite:Mousebite_0.3mm
- added H1: MountingHole, Mousebite:Mousebite_0.3mm, F.Cu at (130.0, 49.4)
- added H2: MountingHole, Mousebite:Mousebite_0.3mm, F.Cu at (130.7, 49.4)
- added H3: MountingHole, Mousebite:Mousebite_0.3mm, F.Cu at (132.0, 49.4)
- added H4: MountingHole, Mousebite:Mousebite_0.3mm, F.Cu at (131.3, 49.4)
Changed lines of the file:
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@@
   )
   (module Mousebite:Mousebite_0.3mm (layer F.Cu)
-    (at 131.97 49.35)
-    (fp_text reference REF** (at 0 0.5) (layer F.SilkS) hide
+    (at 131.33 49.35)
+    (fp_text reference H4 (at 0 0.5) (layer F.SilkS) hide
       (effects (font (size 1 1) (thickness 0.15)))
     )
-    (fp_text value Mousebite_0.3mm (at 0 -0.5) (layer F.Fab) hide
+    (fp_text value MountingHole (at 0 -0.5) (layer F.Fab) hide
       (effects (font (size 1 1) (thickness 0.15)))
     )
@@
   )
   (module Mousebite:Mousebite_0.3mm (layer F.Cu)
-    (at 131.33 49.35)
-    (fp_text reference REF** (at 0 0.5) (layer F.SilkS) hide
+    (at 131.97 49.35)
+    (fp_text reference H3 (at 0 0.5) (layer F.SilkS) hide
       (effects (font (size 1 1) (thickness 0.15)))
     )
-    (fp_text value Mousebite_0.3mm (at 0 -0.5) (layer F.Fab) hide
+    (fp_text value MountingHole (at 0 -0.5) (layer F.Fab) hide
       (effects (font (size 1 1) (thickness 0.15)))
     )
@@
   (module Mousebite:Mousebite_0.3mm (layer F.Cu)
     (at 130.67 49.35)
-    (fp_text reference REF** (at 0 0.5) (layer F.SilkS) hide
+    (fp_text reference H2 (at 0 0.5) (layer F.SilkS) hide
       (effects (font (size 1 1) (thickness 0.15)))
     )
-    (fp_text value Mousebite_0.3mm (at 0 -0.5) (layer F.Fab) hide
+    (fp_text value MountingHole (at 0 -0.5) (layer F.Fab) hide
       (effects (font (size 1 1) (thickness 0.15)))
     )
@@
   (module Mousebite:Mousebite_0.3mm (layer F.Cu)
     (at 130.03 49.35)
-    (fp_text reference REF** (at 0 0.5) (layer F.SilkS) hide
+    (fp_text reference H1 (at 0 0.5) (layer F.SilkS) hide
       (effects (font (size 1 1) (thickness 0.15)))
     )
-    (fp_text value Mousebite_0.3mm (at 0 -0.5) (layer F.Fab) hide
+    (fp_text value MountingHole (at 0 -0.5) (layer F.Fab) hide
       (effects (font (size 1 1) (thickness 0.15)))
     )

Commit message: Add revision indicator
Other:
- board text added: "Rev A"
Changed lines of the file:
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@@
   (general
     (thickness 1.6)
-    (drawings 25)
+    (drawings 26)
     (tracks 118)
     (zones 0)
@@
     )
   )
+  (gr_text "Rev A" (at 134.06 57.28 270) (layer B.SilkS)
+    (effects (font (size 0.8 0.8) (thickness 0.15)) (justify mirror))
+  )
   (gr_text JLCJLCJLCJLC (at 128.8 58.2 90) (layer B.SilkS)

Commit message: Add second GND via to secondary tank capacitors
Routing:
- net GND: track 0.70 -> 2.51 mm, vias 16 -> 18
Changed lines of the file:
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@@
     (thickness 1.6)
     (drawings 26)
-    (tracks 118)
+    (tracks 122)
     (zones 0)
     (modules 23)
@@
   )
   (setup
-    (last_trace_width 0.127)
+    (last_trace_width 0.75)
     (user_trace_width 0.127)
     (user_trace_width 0.25)
@@
   (segment (start 131.63 63.36) (end 131.205736 63.36) (width 0.127) (layer F.Cu) (net 1))
   (segment (start 131.155736 63.31) (end 130.95 63.31) (width 0.127) (layer F.Cu) (net 1))
+  (via (at 134 55.27) (size 0.6) (drill 0.3) (layers F.Cu B.Cu) (net 1))
+  (segment (start 134 56.6) (end 134 55.27) (width 0.75) (layer F.Cu) (net 1))
+  (via (at 128 57.08) (size 0.6) (drill 0.3) (layers F.Cu B.Cu) (net 1))
+  (segment (start 128 56.6) (end 128 57.08) (width 0.75) (layer F.Cu) (net 1))
   (via (at 129.6 62.6) (size 0.6) (drill 0.3) (layers F.Cu B.Cu) (net 2))
   (segment (start 129.6 63.3) (end 129.6 62.6) (width 0.127) (layer F.Cu) (net 2))
